File: Esquema/Analogico.kicad_sch (KiCad schematic)
At the start: 43 parts, among them J1 Conex_bat, J2 Panel Solar, J3 Galga_1, J4 Galga_2, P1 USB_C_Plug_USB2.0, U1 REF3020AIDBZT, U10 NUCLEO-F429ZI, U2 INA826AIDR, U3 TP4057, U4 INA826AIDR, U5 INA826AIDR, U6 XL006, U7 TLV75733PDBV, U8 TLV75733PDBV

Commit message: Placa ya terminada
Signed-off-by: ricardo.socorro <ricardo.socorro@alumnos.upm.es>
Parts:
- J1: footprint Connector_JST:JST_PH_S2B-PH-K_1x02_P2.00mm_Horizontal -> Connector_PinHeader_2.00mm:PinHeader_1x02_P2.00mm_Vertical
Connections:
- net ADC_PESO_1: now also U10.CN7_13 (D22/I2S_B_SD/SPI_B_MOSI); no longer U10.CN9_1 (A0/ADC123_IN3)
- net ADC_PESO_2: now also U10.CN7_17 (D24/SPI_B_NSS); no longer U10.CN9_3 (A1/ADC123_IN10)
- net EN: now also U10.CN10_8 (D4/IO); no longer U10.CN10_13 (D26/IO)
- no-connect marks 91 -> 90
Changed lines of the file:
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@@
 	)
 	(junction
-		(at 101.6 180.34)
-		(diameter 0)
-		(color 0 0 0 0)
-	)
-	(junction
 		(at 149.86 71.12)
 		(diameter 0)
@@
 	)
 	(no_connect
+		(at 436.88 102.87)
+	)
+	(no_connect
 		(at 350.52 95.25)
 	)
@@
 	)
 	(no_connect
-		(at 513.08 85.09)
-	)
-	(no_connect
-		(at 436.88 102.87)
-	)
-	(no_connect
 		(at 416.56 110.49)
 	)
@@
 	)
 	(no_connect
-		(at 594.36 97.79)
-	)
-	(no_connect
-		(at 513.08 87.63)
-	)
-	(no_connect
-		(at 416.56 90.17)
-	)
-	(no_connect
 		(at 594.36 110.49)
 	)
@@
 	)
 	(no_connect
-		(at 436.88 95.25)
-	)
-	(no_connect
 		(at 594.36 80.01)
 	)
@@
 	)
 	(no_connect
+		(at 350.52 69.85)
+	)
+	(no_connect
 		(at 528.32 110.49)
 	)
@@
 	)
 	(no_connect
-		(at 350.52 86.36)
+		(at 436.88 95.25)
 	)
 	(no_connect
@@
 	)
 	(no_connect
+		(at 416.56 90.17)
+	)
+	(no_connect
 		(at 513.08 90.17)
 	)
@@
 	)
 	(no_connect
-		(at 528.32 77.47)
+		(at 594.36 102.87)
 	)
 	(no_connect
-		(at 513.08 92.71)
+		(at 528.32 77.47)
 	)
 	(no_connect
@@
 	)
 	(no_connect
+		(at 350.52 72.39)
+	)
+	(no_connect
 		(at 528.32 105.41)
 	)
@@
 		(at 594.36 82.55)
 	)
+	(no_connect
+		(at 513.08 85.09)
+	)
 	(wire
 		(pts
@@
 	(wire
 		(pts
+			(xy 516.89 92.71) (xy 513.08 92.71)
+		)
+		(stroke
+			(width 0)
+			(type default)
+		)
+	)
+	(wire
+		(pts
 			(xy 515.62 80.01) (xy 513.08 80.01)
 		)
@@
 	(wire
 		(pts
+			(xy 516.89 87.63) (xy 513.08 87.63)
+		)
+		(stroke
+			(width 0)
+			(type default)
+		)
+	)
+	(wire
+		(pts
 			(xy 93.98 48.26) (xy 99.06 48.26)
 		)
@@
 	(wire
 		(pts
-			(xy 347.98 72.39) (xy 350.52 72.39)
-		)
-		(stroke
-			(width 0)
-			(type default)
-		)
-	)
-	(wire
-		(pts
 			(xy 99.06 31.75) (xy 110.49 31.75)
 		)
@@
 	(wire
 		(pts
-			(xy 101.6 180.34) (xy 113.03 180.34)
-		)
-		(stroke
-			(width 0)
-			(type default)
-		)
-	)
-	(wire
-		(pts
 			(xy 173.99 58.42) (xy 173.99 67.31)
 		)
@@
 	(wire
 		(pts
-			(xy 99.06 180.34) (xy 101.6 180.34)
-		)
-		(stroke
-			(width 0)
-			(type default)
-		)
-	)
-	(wire
-		(pts
 			(xy 184.15 58.42) (xy 186.69 58.42)
 		)
@@
 	(wire
 		(pts
-			(xy 598.17 102.87) (xy 594.36 102.87)
-		)
-		(stroke
-			(width 0)
-			(type default)
-		)
-	)
-	(wire
-		(pts
 			(xy 152.4 149.86) (xy 154.94 149.86)
 		)
@@
 	(wire
 		(pts
-			(xy 347.98 69.85) (xy 350.52 69.85)
+			(xy 39.37 31.75) (xy 43.18 31.75)
 		)
 		(stroke
@@
 	(wire
 		(pts
-			(xy 39.37 31.75) (xy 43.18 31.75)
+			(xy 160.02 48.26) (xy 166.37 48.26)
 		)
 		(stroke
@@
 	(wire
 		(pts
-			(xy 160.02 48.26) (xy 166.37 48.26)
+			(xy 101.6 175.26) (xy 107.95 175.26)
 		)
 		(stroke
@@
 	(wire
 		(pts
-			(xy 101.6 175.26) (xy 107.95 175.26)
+			(xy 138.43 147.32) (xy 138.43 149.86)
 		)
 		(stroke
@@
 	(wire
 		(pts
-			(xy 138.43 147.32) (xy 138.43 149.86)
+			(xy 69.85 25.4) (xy 69.85 31.75)
 		)
 		(stroke
@@
 	(wire
 		(pts
-			(xy 69.85 25.4) (xy 69.85 31.75)
+			(xy 166.37 55.88) (xy 166.37 71.12)
 		)
 		(stroke
@@
 	(wire
 		(pts
-			(xy 166.37 55.88) (xy 166.37 71.12)
+			(xy 143.51 118.11) (xy 149.86 118.11)
 		)
 		(stroke
@@
 	(wire
 		(pts
-			(xy 143.51 118.11) (xy 149.86 118.11)
+			(xy 598.17 97.79) (xy 594.36 97.79)
 		)
 		(stroke
@@
 	(wire
 		(pts
+			(xy 101.6 180.34) (xy 113.03 180.34)
+		)
+		(stroke
+			(width 0)
+			(type default)
+		)
+	)
+	(wire
+		(pts
 			(xy 43.18 36.83) (xy 43.18 31.75)
 		)
@@
 		)
 	)
-	(label "ADC_PESO_2"
-		(at 347.98 72.39 180)
-		(effects
-			(font
-				(size 1.27 1.27)
-			)
-			(justify right bottom)
-		)
-	)
 	(label "2.048"
 		(at 596.9 69.85 0)
@@
 		)
 	)
-	(label "ADC_PESO_1"
-		(at 347.98 69.85 180)
-		(effects
-			(font
-				(size 1.27 1.27)
-			)
-			(justify right bottom)
-		)
-	)
 	(label "ADC_V_BAT"
 		(at 179.07 99.06 180)
@@
 		)
 	)
+	(label "EN"
+		(at 598.17 97.79 0)
+		(effects
+			(font
+				(size 1.27 1.27)
+			)
+			(justify left bottom)
+		)
+	)
 	(label "FB"
 		(at 68.58 36.83 180)
@@
 		)
 	)
+	(label "ADC_PESO_1"
+		(at 516.89 92.71 0)
+		(effects
+			(font
+				(size 1.27 1.27)
+			)
+			(justify left bottom)
+		)
+	)
 	(label "2.048"
 		(at 515.62 80.01 0)
@@
 		)
 	)
-	(label "2.048"
-		(at 106.68 133.35 0)
+	(label "ADC_PESO_2"
+		(at 516.89 87.63 0)
 		(effects
 			(font
@@
 		)
 	)
-	(label "EN"
-		(at 598.17 102.87 0)
+	(label "2.048"
+		(at 106.68 133.35 0)
 		(effects
 			(font
@@
 			)
 		)
-		(property "Footprint" "Connector_JST:JST_PH_S2B-PH-K_1x02_P2.00mm_Horizontal"
+		(property "Footprint" "Connector_PinHeader_2.00mm:PinHeader_1x02_P2.00mm_Vertical"
 			(at 154.94 81.28 0)
 			(effects
